File: Charger/Przetwornica/Przetwornica.kicad_sch (KiCad schematic)
At the start: 34 parts, among them U1 XL4015, U2 MCP6001-OT, U3 MCP6001-OT, U4 MCP6001-OT, U5 MCP6001-OT, U6 XL4015

Commit message: next version
Parts:
- removed D2, D3, D5: D, symbol Device:D
- added D2, D3, D6: LL103A, Diode_SMD:D_MiniMELF, symbol Diode:LL42
- C1, C3, C4, C6, C7: value C -> 1uF
- C2, C5, C9: value C_Polarized -> 330uF
- C203: renamed from C8; value C -> 1uF
- D1, D4: value D_Schottky -> B540C-13-F
- L1, L2: value L -> 47uH
- R1, R10: value R -> 9K
- R11, R2: value R -> 1K
- R3: value R -> 100R
- R4: value R -> 4.3K
- R402: renamed from R5; value R -> 820R
- R403: renamed from R6; value R -> 10K
- R404: renamed from R8; value R -> 10K
- R7: value R -> 5.1k
- R9: value R -> 5.1K
Connections:
- net FB: now also D2.1 (K), D3.1 (K), D6.1 (K)
- net Off: now also D3.2 (A)
- net at U5.1: now also D6.2 (A)
- net at R3.1: now also D2.2 (A)
- net Enable renamed +3.3V
Other:
- moved on the sheet: D1, D4, R404, R7

Commit message: Skończone - do przejrzenia
Parts:
- C1, C9: renamed from C2; footprint (none) -> Capacitor_SMD:CP_Elec_10x10
- C10: renamed from C9; footprint (none) -> Capacitor_SMD:CP_Elec_10x10
- C2: renamed from C5; footprint (none) -> Capacitor_SMD:CP_Elec_10x10
- C3: footprint (none) -> Capacitor_SMD:C_0805_2012Metric
- C4: renamed from C6; footprint (none) -> Capacitor_SMD:C_0805_2012Metric
- C5: renamed from C1; footprint (none) -> Capacitor_SMD:C_0805_2012Metric
- C6: renamed from C7; footprint (none) -> Capacitor_SMD:C_0805_2012Metric
- C7: renamed from C4; footprint (none) -> Capacitor_SMD:C_0805_2012Metric
- C8: renamed from C203; footprint (none) -> Capacitor_SMD:C_0805_2012Metric
- D4: renamed from D1; footprint (none) -> Diode_SMD:D_3220_8050Metric_Pad2.65x5.15mm_HandSolder
- D5: renamed from D4; footprint (none) -> Diode_SMD:D_3220_8050Metric_Pad2.65x5.15mm_HandSolder
- L1, L2: footprint (none) -> Inductor_SMD:L_Bourns-SRN8040_8x8.15mm
- R1: renamed from R4; footprint (none) -> Resistor_SMD:R_0805_2012Metric
- R10, R11: footprint (none) -> Resistor_SMD:R_0805_2012Metric
- R2: renamed from R402; footprint (none) -> Resistor_SMD:R_0805_2012Metric
- R3: renamed from R7; footprint (none) -> Resistor_SMD:R_0805_2012Metric
- R4: renamed from R403; footprint (none) -> Resistor_SMD:R_0805_2012Metric
- R5: renamed from R404; footprint (none) -> Resistor_SMD:R_0805_2012Metric
- R6: renamed from R3; footprint (none) -> Resistor_SMD:R_0805_2012Metric
- R7: renamed from R9; footprint (none) -> Resistor_SMD:R_0805_2012Metric
- R8: renamed from R1; footprint (none) -> Resistor_SMD:R_0805_2012Metric
- R9: renamed from R2; footprint (none) -> Resistor_SMD:R_0805_2012Metric
- renumbered D3 to D1, D6 to D3, U3 to U1, U4 to U3, U5 to U4, U1 to U5

Commit message: poprawka
Parts:
- L1, L2: footprint Inductor_SMD:L_Bourns-SRN8040_8x8.15mm -> Inductor_SMD:L_Bourns_SRP1038C_10.0x10.0mm
Changed lines of the file:
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@@
 			)
 		)
-		(property "Footprint" "Inductor_SMD:L_Bourns-SRN8040_8x8.15mm"
+		(property "Footprint" "Inductor_SMD:L_Bourns_SRP1038C_10.0x10.0mm"
 			(at 228.6 62.23 0)
 			(effects
@@
 			)
 		)
-		(property "Footprint" "Inductor_SMD:L_Bourns-SRN8040_8x8.15mm"
+		(property "Footprint" "Inductor_SMD:L_Bourns_SRP1038C_10.0x10.0mm"
 			(at 228.6 110.49 0)
 			(effects
