File: Charger/mcu.kicad_sch (KiCad schematic)
At the start: 0 parts

Commit message: Added Pi Pico model to project
Parts:
- added U23: RaspberryPi_Pico, Module_RaspberryPi_Pico:RaspberryPi_Pico_Common, symbol MCU_Module_RaspberryPi_Pico:RaspberryPi_Pico
Connections:
- new net GND: U23.13 (GND), U23.18 (GND), U23.23 (GND), U23.28 (GND), U23.3 (GND), U23.38 (GND), U23.8 (GND)
Changed lines of the file:
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@@
 	(generator_version "8.0")
 	(paper "A4")
+	(symbol
+		(lib_id "power:GND")
+		(at 146.05 125.73 0)
+		(unit 1)
+		(exclude_from_sim no)
+		(in_bom yes)
+		(on_board yes)
+		(dnp no)
+		(fields_autoplaced yes)
+		(property "Reference" "#PWR063"
+			(at 146.05 132.08 0)
+			(effects
+				(font
+					(size 1.27 1.27)
+				)
+				(hide yes)
+			)
+		)
+		(property "Value" "GND"
+			(at 146.05 130.81 0)
+			(effects
+				(font
+					(size 1.27 1.27)
+				)
+			)
+		)
+		(property "Footprint" ""
+			(at 146.05 125.73 0)
+			(effects
+				(font
+					(size 1.27 1.27)
+				)
+				(hide yes)
+			)
+		)
+		(property "Datasheet" ""
+			(at 146.05 125.73 0)
+			(effects
+				(font
+					(size 1.27 1.27)
+				)
+				(hide yes)
+			)
+		)
+		(property "Description" "Power symbol creates a global label with name \"GND\" , ground"
+			(at 146.05 125.73 0)
+			(effects
+				(font
+					(size 1.27 1.27)
+				)
+				(hide yes)
+			)
+		)
+		(pin "1"
+		)
+		(instances
+			(project "Charger"
+				(path "/f0501846-9b00-4ec1-8596-952177c35a04/8abca69a-4cf1-41f6-b583-47d31555f535"
+					(reference "#PWR063")
+					(unit 1)
+				)
+			)
+		)
+	)
+	(symbol
+		(lib_id "MCU_Module_RaspberryPi_Pico:RaspberryPi_Pico")
+		(at 146.05 87.63 0)
+		(unit 1)
+		(exclude_from_sim no)
+		(in_bom yes)
+		(on_board yes)
+		(dnp no)
+		(fields_autoplaced yes)
+		(property "Reference" "U23"
+			(at 148.2441 124.46 0)
+			(effects
+				(font
+					(size 1.27 1.27)
+				)
+				(justify left)
+			)
+		)
+		(property "Value" "RaspberryPi_Pico"
+			(at 148.2441 127 0)
+			(effects
+				(font
+					(size 1.27 1.27)
+				)
+				(justify left)
+			)
+		)
+		(property "Footprint" "Module_RaspberryPi_Pico:RaspberryPi_Pico_Common"
+			(at 146.05 137.16 0)
+			(effects
+				(font
+					(size 1.27 1.27)
+				)
+				(hide yes)
+			)
+		)
+		(property "Datasheet" "https://datasheets.raspberrypi.com/pico/pico-datasheet.pdf"
+			(at 146.05 139.7 0)
+			(effects
+				(font
+					(size 1.27 1.27)
+				)
+				(hide yes)
+			)
+		)
+		(property "Description" "Versatile and inexpensive microcontroller module (with full pinout for reflow soldering) powered by RP2040 dual-core Arm Cortex-M0+ processor up to 133 MHz, 264kB SRAM, 2MB QSPI flash"
+			(at 146.05 87.63 0)
+			(effects
+				(font
+					(size 1.27 1.27)
+				)
+				(hide yes)
+			)
+		)
+		(pin "22"
+		)
+		(pin "26"
+		)
+		(pin "10"
+		)
+		(pin "12"
+		)
+		(pin "28"
+		)
+		(pin "35"
+		)
+		(pin "37"
+		)
+		(pin "24"
+		)
+		(pin "19"
+		)
+		(pin "5"
+		)
+		(pin "8"
+		)
+		(pin "38"
+		)
+		(pin "15"
+		)
+		(pin "23"
+		)
+		(pin "32"
+		)
+		(pin "29"
+		)
+		(pin "27"
+		)
+		(pin "13"
+		)
+		(pin "11"
+		)
+		(pin "1"
+		)
+		(pin "34"
+		)
+		(pin "4"
+		)
+		(pin "6"
+		)
+		(pin "7"
+		)
+		(pin "36"
+		)
+		(pin "30"
+		)
+		(pin "25"
+		)
+		(pin "31"
+		)
+		(pin "18"
+		)
+		(pin "33"
+		)
+		(pin "9"
+		)
+		(pin "17"
+		)
+		(pin "2"
+		)
+		(pin "3"
+		)
+		(pin "14"
+		)
+		(pin "39"
+		)
+		(pin "40"
+		)
+		(pin "16"
+		)
+		(pin "20"
+		)
+		(pin "21"
+		)
+		(instances
+			(project "Charger"
+				(path "/f0501846-9b00-4ec1-8596-952177c35a04/8abca69a-4cf1-41f6-b583-47d31555f535"
+					(reference "U23")
+					(unit 1)
+				)
+			)
+		)
+	)
 )
