File: Charger/_autosave-mcu.kicad_sch (KiCad schematic)
At the start: 2 parts, among them U23 RaspberryPi_Pico, U24 CD4051B

Commit message: Added connections between uC and other elements
Parts:
- added R72: 10k, symbol Device:R
Connections:
- net BAL_BalV6: now also U24.5 (X5)
- net BAL_BatV1: now also U24.13 (X0)
- net BAL_BatV2: now also U24.14 (X1)
- net BAL_BatV3: now also U24.15 (X2)
- net BAL_BatV4: now also U24.12 (X3)
- net BAL_BatV5: now also U24.1 (X4)
- net BAL_VBal: now also U23.9 (GPIO6)
- net ISENS_EN: now also U23.12 (GPIO9)
- net LOAD_EN: now also U23.10 (GPIO7)
- net LOAD_SetI: now also U23.11 (GPIO8)
- net PSU_Off: now also U23.4 (GPIO2), R72.2
- net PSU_OutV: now also U23.32 (GPIO27_ADC1)
- net PSU_SetI: now also U23.6 (GPIO4)
- net PSU_SetV: now also U23.5 (GPIO3)
- new net +3.3V: R72.1
- no-connect marks 2 -> 5
Other:
- note added: "Do zmiany po dobraniu multipleksera"
