File: Charger/ladowarka.kicad_sch (KiCad schematic)
At the start: 0 parts

Commit message: dodana ladowarka do glownego projektu
drobne zmiany w sumie wszedzie pozbyłem sie 3.3v poza sterowaniem z pinów mcu, dopiescilem rezystorki zby bylo jak najmniej wartości rozszerzylem delikatnie zakres pradowy przetwornicy
Parts:
- added C16, C17, C18, C19, C20, C21: 1uF, symbol Device:C
- added C22, C23, C7, C8: 330uF, symbol Device:C_Polarized
- added D1, D2, D3: LL103A, Diode_SMD:D_MiniMELF, symbol Diode:LL42
- added D4, D5: B540C-13-F, symbol Device:D_Schottky
- added L1, L2: 47uH, symbol Device:L
- added R44, R70: 2k, Resistor_SMD:R_0805_2012Metric_Pad1.20x1.40mm_HandSolder, symbol Device:R
- added R61, R66, R68: 10k, Resistor_SMD:R_0805_2012Metric_Pad1.20x1.40mm_HandSolder, symbol Device:R
- added R62: 5.1k, Resistor_SMD:R_0805_2012Metric_Pad1.20x1.40mm_HandSolder, symbol Device:R
- added R63, R67, R69, R71: 1.2k, Resistor_SMD:R_0805_2012Metric_Pad1.20x1.40mm_HandSolder, symbol Device:R
- added R64, R65: 10K, Resistor_SMD:R_0805_2012Metric_Pad1.20x1.40mm_HandSolder, symbol Device:R
- added U13, U14, U15, U16, U19: MCP6001-OT, Package_TO_SOT_SMD:SOT-23-5, symbol Amplifier_Operational:MCP6001-OT
- added U17, U18: XL4015, Package_TO_SOT_SMD:TO-263-5_TabPin3, symbol Regulator_Switching:XL4015
Connections:
- new net: R70.2, R71.1
- new net: R71.2, U15.1, U16.3 (+)
- new net: D5.1 (K), L2.1, U18.3 (SW)
- new net: D3.2 (A), U16.1
- new net: R64.2, U13.1, U13.4 (-)
- new net: R61.1, R62.2, U13.3 (+)
- new net: R64.1, R70.1, U15.4 (-)
- new net: D2.2 (A), U14.1
- new net: R63.2, R65.1, U15.3 (+)
- new net: C19.2, U18.4 (VC)
- new net: R44.2, R63.1
- new net: D4.1 (K), L1.1, U17.3 (SW)
- new net: R66.1, R67.2, U19.3 (+)
- new net: C18.2, U17.4 (VC)
- new net +5V: R65.2, U13.5 (V+), U14.5 (V+), U15.5 (V+), U16.5 (V+), U19.5 (V+)
- new net FB: D1.1 (K), D2.1 (K), D3.1 (K), U17.2 (FB), U18.2 (FB)
- new net GND: C16.2, C17.2, C20.2, C21.2, C22.2, C23.2, C7.2, C8.2, D4.2 (A), D5.2 (A), R44.1, R62.1, R67.1, R69.2, U13.2 (V-), U14.2 (V-), U15.2 (V-), U16.2 (V-), U17.1 (GND), U18.1 (GND), U19.2 (V-)
- new net Hall: U16.4 (-)
- new net Off: D1.2 (A)
- new net Ref: R68.2, R69.1, U14.3 (+)
- new net Set I: R61.2
- new net Set V: U14.4 (-)
- new net V_OUT (ADC): U19.1, U19.4 (-)
- new net Vin: C16.1, C17.1, C18.1, C19.1, C7.1, C8.1, U17.5 (VIN), U18.5 (VIN)
- new net Vout: C20.1, C21.1, C22.1, C23.1, L1.2, L2.2, R66.2, R68.1

Commit message: dodanie sekcji zasilacza
i dodanie footprintów prawie wszedzie
Parts:
- C16, C17, C18, C19, C20, C21: footprint (none) -> Capacitor_SMD:C_0805_2012Metric_Pad1.18x1.45mm_HandSolder
Changed lines of the file:
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@@
 			)
 		)
-		(property "Footprint" ""
+		(property "Footprint" "Capacitor_SMD:C_0805_2012Metric_Pad1.18x1.45mm_HandSolder"
 			(at 244.8052 68.58 0)
 			(effects
@@
 			)
 		)
-		(property "Footprint" ""
+		(property "Footprint" "Capacitor_SMD:C_0805_2012Metric_Pad1.18x1.45mm_HandSolder"
 			(at 187.6552 107.95 0)
 			(effects
@@
 			)
 		)
-		(property "Footprint" ""
+		(property "Footprint" "Capacitor_SMD:C_0805_2012Metric_Pad1.18x1.45mm_HandSolder"
 			(at 233.3752 116.84 0)
 			(effects
@@
 			)
 		)
-		(property "Footprint" ""
+		(property "Footprint" "Capacitor_SMD:C_0805_2012Metric_Pad1.18x1.45mm_HandSolder"
 			(at 182.5752 116.84 0)
 			(effects
@@
 			)
 		)
-		(property "Footprint" ""
+		(property "Footprint" "Capacitor_SMD:C_0805_2012Metric_Pad1.18x1.45mm_HandSolder"
 			(at 182.5752 68.58 0)
 			(effects
@@
 			)
 		)
-		(property "Footprint" ""
+		(property "Footprint" "Capacitor_SMD:C_0805_2012Metric_Pad1.18x1.45mm_HandSolder"
 			(at 187.6552 59.69 0)
 			(effects

Commit message: drobne zmiany
Parts:
- C22, C23, C7, C8: value 330uF -> 470u; footprint (none) -> Library:CP_Elec_12.5x13.5
- D4, D5: value B540C-13-F -> B540C; footprint (none) -> Diode_SMD:D_3220_8050Metric_Pad2.65x5.15mm_HandSolder
- L1, L2: footprint (none) -> Inductor_SMD:L_Bourns_SRP1038C_10.0x10.0mm
Connections:
- net Vin: now also C23.1; no longer C8.1
- net Vout: now also C8.1; no longer C23.1
Other:
- moved on the sheet: C16, C17, C18, C19, D4, D5, R69

Commit message: pcb up
Parts:
- removed U13, U14, U15, U16: MCP6001-OT, Package_TO_SOT_SMD:SOT-23-5, symbol Amplifier_Operational:MCP6001-OT
- added C12, C13: 100n, Capacitor_SMD:C_0805_2012Metric_Pad1.18x1.45mm_HandSolder, symbol Device:C
- added U25: MCP6004, Package_SO:SOIC-14_3.9x8.7mm_P1.27mm, symbol Amplifier_Operational:MCP6004
Connections:
- net +5V: now also C12.1, C13.1, U25.4 (V+)
- net GND: now also C12.2, C13.2, U25.11 (V-)
- net Hall: now also U25.9 (-)
- net Ref: now also U25.12 (+)
- net Set V: now also U25.13 (-)
- net at R71.2: now also U25.10 (+), U25.7
- net at D3.2 (A): now also U25.8
- net at R64.2: now also U25.1, U25.2 (-)
- net at R61.1, R62.2: now also U25.3 (+)
- net at R64.1, R70.1: now also U25.6 (-)
- net at D2.2 (A): now also U25.14
- net at R63.2, R65.1: now also U25.5 (+)

Commit message: pcb poukladane
usuniete 3 kondensatory
brak poligonow i odprowadzania ciepla
Parts:
- removed C23, C7, C8: 470u, Library:CP_Elec_12.5x13.5, symbol Device:C_Polarized
Changed lines of the file:
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@@
-	)
-	(symbol
-		(lib_id "Device:C_Polarized")
-		(at 251.46 64.77 0)
-		(unit 1)
-		(exclude_from_sim no)
-		(in_bom yes)
-		(on_board yes)
-		(dnp no)
-		(property "Reference" "C8"
-			(at 254 63.246 0)
-			(effects
-				(font
-					(size 1.27 1.27)
-				)
-				(justify left)
-			)
-		)
-		(property "Value" "470u"
-			(at 254 65.786 0)
-			(effects
-				(font
-					(size 1.27 1.27)
-				)
-				(justify left)
-			)
-		)
-		(property "Footprint" "Library:CP_Elec_12.5x13.5"
-			(at 252.4252 68.58 0)
-			(effects
-				(font
-					(size 1.27 1.27)
-				)
-				(hide yes)
-			)
-		)
-		(property "Datasheet" "~"
-			(at 251.46 64.77 0)
-			(effects
-				(font
-					(size 1.27 1.27)
-				)
-				(hide yes)
-			)
-		)
-		(property "Description" "Polarized capacitor"
-			(at 251.46 64.77 0)
-			(effects
-				(font
-					(size 1.27 1.27)
-				)
-				(hide yes)
-			)
-		)
-		(pin "2"
-		)
-		(pin "1"
-		)
-		(instances
-			(project "Charger"
-				(path "/f0501846-9b00-4ec1-8596-952177c35a04/b3aae3c9-c46d-4aed-bc70-e41b62c2dce3"
-					(reference "C8")
-					(unit 1)
-				)
-			)
-		)
 	)
 	(symbol
@@
 					(unit 1)
 				)
-			)
-		)
-	)
-	(symbol
-		(lib_id "Device:C_Polarized")
-		(at 173.99 64.77 0)
-		(unit 1)
-		(exclude_from_sim no)
-		(in_bom yes)
-		(on_board yes)
-		(dnp no)
-		(property "Reference" "C7"
-			(at 176.53 63.246 0)
-			(effects
-				(font
-					(size 1.27 1.27)
-				)
-				(justify left)
-			)
-		)
-		(property "Value" "470u"
-			(at 176.53 65.786 0)
-			(effects
-				(font
-					(size 1.27 1.27)
-				)
-				(justify left)
-			)
-		)
-		(property "Footprint" "Library:CP_Elec_12.5x13.5"
-			(at 174.9552 68.58 0)
-			(effects
-				(font
-					(size 1.27 1.27)
-				)
-				(hide yes)
-			)
-		)
-		(property "Datasheet" "~"
-			(at 173.99 64.77 0)
-			(effects
-				(font
-					(size 1.27 1.27)
-				)
-				(hide yes)
-			)
-		)
-		(property "Description" "Polarized capacitor"
-			(at 173.99 64.77 0)
-			(effects
-				(font
-					(size 1.27 1.27)
-				)
-				(hide yes)
-			)
-		)
-		(pin "2"
-		)
-		(pin "1"
-		)
-		(instances
-			(project "Charger"
-				(path "/f0501846-9b00-4ec1-8596-952177c35a04/b3aae3c9-c46d-4aed-bc70-e41b62c2dce3"
-					(reference "C7")
-					(unit 1)
-				)
-			)
-		)
-	)
-	(symbol
-		(lib_id "Device:C_Polarized")
-		(at 173.99 113.03 0)
-		(unit 1)
-		(exclude_from_sim no)
-		(in_bom yes)
-		(on_board yes)
-		(dnp no)
-		(property "Reference" "C23"
-			(at 176.53 111.506 0)
-			(effects
-				(font
-					(size 1.27 1.27)
-				)
-				(justify left)
-			)
-		)
-		(property "Value" "470u"
-			(at 176.53 114.046 0)
-			(effects
-				(font
-					(size 1.27 1.27)
-				)
-				(justify left)
-			)
-		)
-		(property "Footprint" "Library:CP_Elec_12.5x13.5"
-			(at 174.9552 116.84 0)
-			(effects
-				(font
-					(size 1.27 1.27)
-				)
-				(hide yes)
-			)
-		)
-		(property "Datasheet" "~"
-			(at 173.99 113.03 0)
-			(effects
-				(font
-					(size 1.27 1.27)
-				)
-				(hide yes)
-			)
-		)
-		(property "Description" "Polarized capacitor"
-			(at 173.99 113.03 0)
-			(effects
-				(font
-					(size 1.27 1.27)
-				)
-				(hide yes)
-			)
-		)
-		(pin "2"
-		)
-		(pin "1"
-		)
-		(instances
-			(project "Charger"
-				(path "/f0501846-9b00-4ec1-8596-952177c35a04/b3aae3c9-c46d-4aed-bc70-e41b62c2dce3"
-					(reference "C23")
-					(unit 1)
-				)

Commit message: poprawki hardware
Other:
- note added: "r44 i r70 2.2k"
- note added: "r62 wydupcyć"
Changed lines of the file:
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@@
+		)
+	)
+	(text "r44 i r70 2.2k\n"
+		(exclude_from_sim no)
+		(at 92.71 34.036 0)
+		(effects
+			(font
+				(size 1.27 1.27)
+			)
+		)
+	)
+	(text "r62 wydupcyć"
+		(exclude_from_sim no)
+		(at 31.242 62.484 0)
+		(effects
+			(font
+				(size 1.27 1.27)
+			)
 		)
 	)
